Commit message: ur5e to init, usd ok

File: assets/ur5e/ur.urdf.xacro (robot description, xacro)
@@ -9,5 +9,5 @@
   <!-- possible 'ur_type' values: ur3, ur3e, ur5, ur5e, ur7e, ur10, ur10e, ur12e, ur16e, ur8long, ur15, ur18, ur20, ur30 -->
   <!-- the default value should raise an error in case this was called without defining the type -->
-  <xacro:arg name="ur_type" default="urXe"/>
+  <xacro:arg name="ur_type" default="ur5e"/>
   <!-- parameters -->
   <xacro:arg name="tf_prefix" default="" />

File: assets/ur5e/ur5e.urdf (robot description, URDF)
Before this commit: robot ur5e_robot, 11 links, 10 joints
Links:
- link base_link_inertia: geometry collision mesh filename=/home/user/Documents/RL_Arm/assets/ur5e/collisions/base.stl; visual mesh filename=/home/user/Documents/RL_Arm/assets/ur5e/visuals/base.dae
- link forearm_link: geometry collision mesh filename=/home/user/Documents/RL_Arm/assets/ur5e/collisions/forearm.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; visual mesh filename=/home/user/Documents/RL_Arm/assets/ur5e/visuals/forearm.dae
- link shoulder_link: geometry collision mesh filename=/home/user/Documents/RL_Arm/assets/ur5e/collisions/shoulder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; visual mesh filename=/home/user/Documents/RL_Arm/assets/ur5e/visuals/shoulder.dae
- link upper_arm_link: geometry collision mesh filename=/home/user/Documents/RL_Arm/assets/ur5e/collisions/upperarm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; visual mesh filename=/home/user/Documents/RL_Arm/assets/ur5e/visuals/upperarm.dae
- link wrist_1_link: geometry collision mesh filename=/home/user/Documents/RL_Arm/assets/ur5e/collisions/wrist1.s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; visual mesh filename=/home/user/Documents/RL_Arm/assets/ur5e/visuals/wrist1.dae
- link wrist_2_link: geometry collision mesh filename=/home/user/Documents/RL_Arm/assets/ur5e/collisions/wrist2.s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; visual mesh filename=/home/user/Documents/RL_Arm/assets/ur5e/visuals/wrist2.dae
- link wrist_3_link: geometry collision mesh filename=/home/user/Documents/RL_Arm/assets/ur5e/collisions/wrist3.s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; visual mesh filename=/home/user/Documents/RL_Arm/assets/ur5e/visuals/wrist3.dae
